File: Electronics/DumbBadge.sch (EAGLE design)
At the start: 124 parts, among them J1 40PINFPCM4-1734839-0, SW1 SPST_TACT-KMR2, U1 RA8875, U5 74HC4050, U6 MAX3232, U7 TPS61090RSAR, U8 MCP73831T-2ACI/OT, X2 FH12-50S-0.5SH, X4 32.768, Y1 20MHz

Commit message: push
Parts:
- removed C1, C10, C11, C12, C4, C5, C6, C7, C8, C9: 0.1uF, microbuilder:CAP_CERAMIC0805-NOOUTLINE
- removed C2, C3: 20pF, microbuilder:CAP_CERAMIC0805-NOOUTLINE
- removed J1: 40PINFPCM4-1734839-0, adafruit:40PINFPCM4-1734839-0
- removed JP2: Breakout, adafruit:PINHD-1X15-CB
- removed L: RED, microbuilder:LED0805_NOOUTLINE
- removed R12: 10K, microbuilder:RESISTOR0805_NOOUTLINE
- removed R2: 2.2K, microbuilder:RESISTOR_0603_NOOUT
- removed R3: 1M, microbuilder:RESISTOR0805_NOOUTLINE
- removed R4, R5, R6, R7, R8: 33, microbuilder:RESISTOR_4PACK_US
- removed U1: RA8875, microbuilder:RA8875
- removed U5: 74HC4050, microbuilder:74HC4050D
- removed X2: FH12-50S-0.5SH, con-hirose:FH12-50S-0.5SH
- removed Y1: 20MHz, microbuilder:CRYSTAL3.2X2.5
Connections:
- removed net +24V: J1-2.MS
- removed net 1: X2-13.1, X2-14.1, X2-15.1, X2-16.1, X2-17.1, X2-18.1, X2-19.1, X2-20.1, X2-21.1, X2-22.1, X2-23.1, X2-24.1, X2-25.1, X2-26.1, X2-27.1, X2-28.1, X2-29.1, X2-30.1, X2-31.1, X2-32.1, X2-33.1, X2-34.1, X2-35.1, X2-36.1
- removed net 1.5V: C10.1, C12.1, C8.1, C9.1, U1.CORE_VDD@1, U1.CORE_VDD@2, U1.CORE_VDD@3, U1.LDO_OUT, U1.OSC_VDD
- removed net B3: J1-24.MS, R4G$4.2
- removed net B4: J1-25.MS, R4G$3.2
- removed net B5: J1-26.MS, R4G$2.2
- removed net B6: J1-27.MS, R4G$1.2
- removed net B7: J1-28.MS, R5G$4.2
- removed net CS: JP2.8, X2-42.1
- removed net CS_BUFFER: U5.3A
- removed net D/C: X2-41.1
- removed net DE: J1-34.MS, R8G$1.2, X2-12.1
- removed net DOTCLK: X2-11.1
- removed net G2: J1-15.MS, R5G$3.2
- removed net G3: J1-16.MS, R5G$2.2
- removed net G4: J1-17.MS, R5G$1.2
- removed net G5: J1-18.MS, R6G$4.2
- removed net G6: J1-19.MS, R6G$3.2
- removed net G7: J1-20.MS, R6G$2.2
- removed net HSYNC: J1-32.MS, R8G$4.2, X2-10.1
- removed net IM0: X2-4.1
- removed net IM1: X2-5.1
- removed net IM2: X2-6.1
- removed net IM3: X2-7.1
- removed net INT: JP2.5, U1.INT#
- removed net LEDA: X2-1.1
- removed net LEDK: J1-1.MSV
- removed net LEDK1: X2-2.1
- removed net LEDK2: X2-3.1
- removed net MOSI_3V: U1.SDI/SDA, U5.2Y
- removed net MOSI_BUFFER: U5.2A
- removed net N$23: R4G$4.1, U1.PDAT0
- removed net N$25: R4G$3.1, U1.PDAT1
- removed net N$27: R4G$2.1, U1.PDAT2
- removed net N$28: R4G$1.1, U1.PDAT3
- removed net N$29: R5G$4.1, U1.PDAT4
- removed net N$30: R5G$3.1, U1.PDAT5
- removed net N$31: R5G$2.1, U1.PDAT6
- removed net N$32: R5G$1.1, U1.PDAT7
- removed net N$33: R6G$4.1, U1.PDAT8
- removed net N$34: R6G$3.1, U1.PDAT9
- removed net N$35: R6G$2.1, U1.PDAT10
- removed net N$36: R6G$1.1, U1.PDAT11
- removed net N$37: R7G$4.1, U1.PDAT12
- removed net N$38: R7G$3.1, U1.PDAT13
- removed net N$39: R7G$2.1, U1.PDAT14
- removed net N$40: R7G$1.1, U1.PDAT15
- removed net N$41: R8G$1.1, U1.DE
- removed net N$42: R8G$2.1, U1.PCLK
- removed net N$43: R8G$3.1, U1.VSYNC
- removed net N$44: R8G$4.1, U1.HSYNC
- removed net N$45: C1.1, U1.ADC_VREF
- removed net N$46: C2.2, R3.2, U1.XI, Y1.2
- removed net N$47: C3.2, R3.1, U1.XO, Y1.1
- removed net N$48: L.A, R2.2
- removed net ON/OFF: J1-31.MS, U1.GPOX
- removed net PIXCLK: J1-30.MS, R8G$2.2
- removed net PWM0: U1.PWM1
- removed net R3: J1-8.MS, R6G$1.2
- removed net R4: J1-9.MS, R7G$4.2
- removed net R5: J1-10.MS, R7G$3.2
- removed net R6: J1-11.MS, R7G$2.2
- removed net R7: J1-12.MS, R7G$1.2
- removed net RD: X2-39.1
- removed net RESET: JP2.7, X2-8.1
- removed net RESET_3V: U1.RST#, U5.4Y
- removed net RESET_BUFFER: R12.1, U5.4A
- removed net SCK_BUFFER: U5.1A
- removed net SDI: X2-38.1
- removed net SDO: X2-37.1
- removed net SPI_CLK_3V: U1.SCL, U5.1Y
- removed net SPI_CS_3V: U1.SCS#, U5.3Y
- removed net VCC: X2-44.1
- removed net VDDI: X2-43.1
- removed net VIN: JP2.15
- removed net VSYNC: J1-33.MS, R8G$3.2, X2-9.1
- removed net WAIT: JP2.6, U1.WAIT#
- removed net WR: X2-40.1
- removed net X+: J1-37.MS
- removed net X-: J1-39.MS
- removed net XL: X2-48.1
- removed net XR: X2-46.1
- removed net Y+: J1-38.MS
- removed net Y-: J1-40.MS
- removed net YD: X2-47.1
- removed net YU: X2-49.1
- net +3V3: no longer C11.1, C4.1, C5.1, C6.1, C7.1, J1-4.MS, JP2.13, R12.2, U1.ADC_VDD, U1.CS#, U1.OSC_VDDP, U1.PS, U1.RD#/EN, U1.RS, U1.SIFS1, U1.VDDP@1, U1.VDDP@2, U1.VDDP@3, U1.VDDP@4, U1.WR#/RW#, U5.VCC
- net D13: no longer R2.1
- net GND: no longer C1.2, C10.2, C11.2, C12.2, C2.1, C3.1, C4.2, C5.2, C6.2, C7.2, C8.2, C9.2, J1-13.MS, J1-14.MS, J1-21.MS, J1-22.MS, J1-23.MS, J1-29.MS, J1-3.MS, J1-36.MS, J1-5.MS, J1-6.MS, J1-7.MS, JP2.14, L.C, U1.ADC_GND, U1.C86, U1.GND@1, U1.GND@2, U1.GND@3, U1.GND@4, U1.GPIX, U1.IICA0, U1.IICA1, U1.KIN0/GPI0, U1.KIN1/GPI1, U1.KIN2/GPI2, U1.KIN3/GPI3, U1.KIN4/GPI4, U1.LDO_GND, U1.OSC_GND, U1.OSC_GNDP, U1.SIFS0, U1.TEST0, U1.TEST1, U1.TEST2, U5.GND, X2-45.1, X2-50.1
- net MISO: no longer JP2.10, U1.SDO
- net MOSI: no longer JP2.9
- net SCK: no longer JP2.11
Other:
- note removed: "BREAKOUTS"
- note removed: "RED LED"
