File: Electronics/DumbBadgeFusion.sch (EAGLE design)
At the start: 139 parts, among them IC1 74245MTC, IC2 74245MTC, IC3 74245MTC, SW1 SPST_TACT-KMR2, T1 MMUN2133LT1G, U1 TDP3E001DRLR-SOT-23-5SOT-23-5, U2 TPS61090RSAR, U3 MCP73871, U4 FAN5333BSX, U6 MAX3232, X4 32.768

Commit message: redid and prettified power supply
Parts:
- removed LED2: BLUE, microbuilder:LED0805_NOOUTLINE
- removed NCP21XW153J03RA: 15K, microbuilder:RESISTOR0805_NOOUTLINE
- added C13, C14: 1.0uF, SparkFun-Capacitors:1.0UF-0603-16V-10%
- added U5: ADP160AUJZ-1.8-R7, SparkFun-IC-Power:ADP160
- C5: value 100uF -> 1.0uF; device rcl:C-USC1210 -> SparkFun-Capacitors:1.0UF-0603-16V-10%
- R5: value 1K -> NCP21XW153J03RA
- renumbered CHRG/LBO to BATT_LOW
Connections:
- removed net N$9: LED2.A, R5.2
- new net 1.8V: C14.1, U5.VOUT
- net 5.0V: now also C13.1, U5.EN, U5.VIN; no longer R5.1
- net GND: now also C13.2, C14.2, R5.1, U5.GND; no longer LED2.C, NCP21XW153J03RA.1
- net N$14: now also R5.2; no longer NCP21XW153J03RA.2
Other:
- moved on the sheet: K-5, K_4, K_6, K_7, K_8, K_9, K_B, K_C, K_D, K_E, K_F, K_G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

Commit message: lots of updating
Parts:
- removed C13: 1.0uF, SparkFun-Capacitors:1.0UF-0603-16V-10%
- removed U5: ADP160AUJZ-1.8-R7, SparkFun-IC-Power:ADP160
- added R15: 1K, microbuilder:RESISTOR0805_NOOUTLINE
- added R18: 1.2K, microbuilder:RESISTOR0805_NOOUTLINE
- added TP10, TP9: TPB1,27, testpad:TPB1,27
- renumbered B2 to B1
Connections:
- net 1.8V: now also R15.1, R18.2, TP9.TP; no longer U5.VOUT
- net 3V3: now also R15.2
- net 5.0V: no longer C13.1, U5.EN, U5.VIN
- net GND: now also R18.1, TP10.TP; no longer C13.2, U5.GND
Other:
- moved on the sheet: C14

Commit message: modified models
Parts:
- added TP11, TP12, TP13, TP14, TP15, TP16: TPB1,27, testpad:TPB1,27
Other:
- note added: "We don't expect to put anything except for 1.8V serial level shifters on this rail, so it just gets a voltage divider. If better regulation is required, R15 and R18 should be < 1% resistors"
- moved on the sheet: C14, R15, R18, TP9
Changed lines of the file:
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@@
 <part name="TP9" library="testpad" library_urn="urn:adsk.eagle:library:385" deviceset="TP" device="B1,27" package3d_urn="urn:adsk.eagle:package:27944/2"/>
 <part name="TP10" library="testpad" library_urn="urn:adsk.eagle:library:385" deviceset="TP" device="B1,27" package3d_urn="urn:adsk.eagle:package:27944/2"/>
+<part name="TP11" library="testpad" library_urn="urn:adsk.eagle:library:385" deviceset="TP" device="B1,27" package3d_urn="urn:adsk.eagle:package:27944/2"/>
+<part name="TP12" library="testpad" library_urn="urn:adsk.eagle:library:385" deviceset="TP" device="B1,27" package3d_urn="urn:adsk.eagle:package:27944/2"/>
+<part name="TP13" library="testpad" library_urn="urn:adsk.eagle:library:385" deviceset="TP" device="B1,27" package3d_urn="urn:adsk.eagle:package:27944/2"/>
+<part name="TP14" library="testpad" library_urn="urn:adsk.eagle:library:385" deviceset="TP" device="B1,27" package3d_urn="urn:adsk.eagle:package:27944/2"/>
+<part name="TP15" library="testpad" library_urn="urn:adsk.eagle:library:385" deviceset="TP" device="B1,27" package3d_urn="urn:adsk.eagle:package:27944/2"/>
+<part name="TP16" library="testpad" library_urn="urn:adsk.eagle:library:385" deviceset="TP" device="B1,27" package3d_urn="urn:adsk.eagle:package:27944/2"/>
 </parts>
 <sheets>
@@
 <attribute name="SHEET" x="200.66" y="6.35" size="2.54" layer="94" font="vector"/>
 </instance>
+<instance part="TP11" gate="G$1" x="10.16" y="180.34" smashed="yes">
+<attribute name="NAME" x="8.89" y="181.61" size="1.778" layer="95"/>
+<attribute name="TP_SIGNAL_NAME" x="11.43" y="179.07" size="1.778" layer="97"/>
+</instance>
+<instance part="TP12" gate="G$1" x="15.24" y="180.34" smashed="yes">
+<attribute name="NAME" x="13.97" y="181.61" size="1.778" layer="95"/>
+<attribute name="TP_SIGNAL_NAME" x="16.51" y="179.07" size="1.778" layer="97"/>
+</instance>
+<instance part="TP13" gate="G$1" x="20.32" y="180.34" smashed="yes">
+<attribute name="NAME" x="19.05" y="181.61" size="1.778" layer="95"/>
+<attribute name="TP_SIGNAL_NAME" x="21.59" y="179.07" size="1.778" layer="97"/>
+</instance>
+<instance part="TP14" gate="G$1" x="25.4" y="180.34" smashed="yes">
+<attribute name="NAME" x="24.13" y="181.61" size="1.778" layer="95"/>
+<attribute name="TP_SIGNAL_NAME" x="26.67" y="179.07" size="1.778" layer="97"/>
+</instance>
+<instance part="TP15" gate="G$1" x="30.48" y="180.34" smashed="yes">
+<attribute name="NAME" x="29.21" y="181.61" size="1.778" layer="95"/>
+<attribute name="TP_SIGNAL_NAME" x="31.75" y="179.07" size="1.778" layer="97"/>
+</instance>
+<instance part="TP16" gate="G$1" x="35.56" y="180.34" smashed="yes">
+<attribute name="NAME" x="34.29" y="181.61" size="1.778" layer="95"/>
+<attribute name="TP_SIGNAL_NAME" x="36.83" y="179.07" size="1.778" layer="97"/>
+</instance>
 </instances>
 <busses>
@@
 <text x="152.4" y="177.8" size="6.4516" layer="94">Battery Charging</text>
 <text x="5.08" y="177.8" size="6.4516" layer="94">5 V Switching Reg</text>
+<text x="172.974" y="196.596" size="1.778" layer="97">We don't expect to put anything
+except for 1.8V serial level shifters
+on this rail, so it just gets a voltage
+divider.
+If better regulation is required, R15
+and R18 should be &lt; 1% resistors</text>
 </plain>
 <instances>
@@
 <attribute name="VALUE" x="258.064" y="213.741" size="1.778" layer="96" font="vector"/>
 </instance>
-<instance part="C14" gate="G$1" x="180.34" y="208.28" smashed="yes">
-<attribute name="NAME" x="181.864" y="211.201" size="1.778" layer="95" font="vector"/>
-<attribute name="VALUE" x="181.864" y="206.121" size="1.778" layer="96" font="vector"/>
-</instance>
-<instance part="SUPPLY3" gate="G$1" x="180.34" y="218.44" smashed="yes">
-<attribute name="VALUE" x="180.34" y="221.234" size="1.778" layer="96" align="bottom-center"/>
-</instance>
-<instance part="GND16" gate="1" x="180.34" y="200.914" smashed="yes">
-<attribute name="VALUE" x="177.8" y="198.374" size="1.778" layer="96"/>
-</instance>
-<instance part="R15" gate="G$1" x="172.72" y="223.52" smashed="yes" rot="R90">
-<attribute name="NAME" x="170.18" y="223.52" size="1.27" layer="95" font="vector" rot="R90" align="center"/>
-<attribute name="VALUE" x="172.72" y="223.52" size="1.016" layer="96" font="vector" ratio="15" rot="R90" align="center"/>
-</instance>
-<instance part="R18" gate="G$1" x="172.72" y="208.28" smashed="yes" rot="R90">
-<attribute name="NAME" x="170.18" y="208.28" size="1.27" layer="95" font="vector" rot="R90" align="center"/>
-<attribute name="VALUE" x="172.72" y="208.28" size="1.016" layer="96" font="vector" ratio="15" rot="R90" align="center"/>
-</instance>
-<instance part="U$12" gate="G$1" x="172.72" y="236.22" smashed="yes">
-<attribute name="VALUE" x="171.196" y="237.236" size="1.27" layer="96"/>
-</instance>
-<instance part="TP9" gate="G$1" x="187.96" y="218.44" smashed="yes">
-<attribute name="NAME" x="186.69" y="219.71" size="1.778" layer="95"/>
-<attribute name="TP_SIGNAL_NAME" x="189.23" y="217.17" size="1.778" layer="97"/>
+<instance part="C14" gate="G$1" x="162.56" y="210.82" smashed="yes">
+<attribute name="NAME" x="164.084" y="213.741" size="1.778" layer="95" font="vector"/>
+<attribute name="VALUE" x="164.084" y="208.661" size="1.778" layer="96" font="vector"/>
+</instance>
+<instance part="SUPPLY3" gate="G$1" x="162.56" y="220.98" smashed="yes">
+<attribute name="VALUE" x="162.56" y="223.774" size="1.778" layer="96" align="bottom-center"/>
+</instance>
+<instance part="GND16" gate="1" x="162.56" y="203.454" smashed="yes">
+<attribute name="VALUE" x="160.02" y="200.914" size="1.778" layer="96"/>
+</instance>
+<instance part="R15" gate="G$1" x="154.94" y="226.06" smashed="yes" rot="R90">
+<attribute name="NAME" x="152.4" y="226.06" size="1.27" layer="95" font="vector" rot="R90" align="center"/>
+<attribute name="VALUE" x="154.94" y="226.06" size="1.016" layer="96" font="vector" ratio="15" rot="R90" align="center"/>
+</instance>
+<instance part="R18" gate="G$1" x="154.94" y="210.82" smashed="yes" rot="R90">
+<attribute name="NAME" x="152.4" y="210.82" size="1.27" layer="95" font="vector" rot="R90" align="center"/>
+<attribute name="VALUE" x="154.94" y="210.82" size="1.016" layer="96" font="vector" ratio="15" rot="R90" align="center"/>
+</instance>
+<instance part="U$12" gate="G$1" x="154.94" y="238.76" smashed="yes">
+<attribute name="VALUE" x="153.416" y="239.776" size="1.27" layer="96"/>
+</instance>
+<instance part="TP9" gate="G$1" x="170.18" y="220.98" smashed="yes">
+<attribute name="NAME" x="168.91" y="222.25" size="1.778" layer="95"/>
+<attribute name="TP_SIGNAL_NAME" x="171.45" y="219.71" size="1.778" layer="97"/>
 </instance>
 <instance part="TP10" gate="G$1" x="182.88" y="111.76" smashed="yes">
@@
 <pinref part="R16" gate="G$1" pin="1"/>
 <pinref part="GND11" gate="1" pin="GND"/>
+<pinref part="TP10" gate="G$1" pin="TP"/>
+<wire x1="193.04" y1="109.22" x2="182.88" y2="109.22" width="0.1524" layer="91"/>
+<label x="184.912" y="109.474" size="1.778" layer="95"/>
 </segment>
 <segment>
@@
 <segment>
 <pinref part="C14" gate="G$1" pin="2"/>
-<wire x1="180.34" y1="205.74" x2="180.34" y2="203.454" width="0.1524" layer="91"/>
+<wire x1="162.56" y1="208.28" x2="162.56" y2="205.994" width="0.1524" layer="91"/>
 <pinref part="GND16" gate="1" pin="GND"/>
-<wire x1="180.34" y1="203.454" x2="180.34" y2="203.2" width="0.1524" layer="91"/>
-<wire x1="180.34" y1="203.2" x2="180.34" y2="203.454" width="0.1524" layer="91"/>
+<wire x1="162.56" y1="205.994" x2="162.56" y2="205.74" width="0.1524" layer="91"/>
+<wire x1="162.56" y1="205.74" x2="162.56" y2="205.994" width="0.1524" layer="91"/>
 <pinref part="R18" gate="G$1" pin="1"/>
-<wire x1="172.72" y1="203.2" x2="180.34" y2="203.2" width="0.1524" layer="91"/>
-<wire x1="180.34" y1="203.2" x2="180.34" y2="203.454" width="0.1524" layer="91"/>
-<junction x="180.34" y="203.454"/>
-</segment>
-<segment>
-<pinref part="TP10" gate="G$1" pin="TP"/>
-<wire x1="193.04" y1="109.22" x2="182.88" y2="109.22" width="0.1524" layer="91"/>
-<label x="184.912" y="109.474" size="1.778" layer="95"/>
+<wire x1="154.94" y1="205.74" x2="162.56" y2="205.74" width="0.1524" layer="91"/>
+<wire x1="162.56" y1="205.74" x2="162.56" y2="205.994" width="0.1524" layer="91"/>
+<junction x="162.56" y="205.994"/>
 </segment>
 </net>
@@
 <segment>
 <pinref part="U$12" gate="G$1" pin="5.0V"/>
-<wire x1="172.72" y1="228.6" x2="172.72" y2="233.68" width="0.1524" layer="91"/>
+<wire x1="154.94" y1="231.14" x2="154.94" y2="236.22" width="0.1524" layer="91"/>
 <pinref part="R15" gate="G$1" pin="2"/>
 </segment>
@@
 <pinref part="C14" gate="G$1" pin="1"/>
 <pinref part="SUPPLY3" gate="G$1" pin="1.8V"/>
-<wire x1="180.34" y1="218.44" x2="180.34" y2="215.9" width="0.1524" layer="91"/>
+<wire x1="162.56" y1="220.98" x2="162.56" y2="218.44" width="0.1524" layer="91"/>
 <pinref part="R15" gate="G$1" pin="1"/>
-<wire x1="180.34" y1="215.9" x2="180.34" y2="213.36" width="0.1524" layer="91"/>
-<wire x1="172.72" y1="218.44" x2="172.72" y2="215.9" width="0.1524" layer="91"/>
-<wire x1="172.72" y1="215.9" x2="180.34" y2="215.9" width="0.1524" layer="91"/>
-<junction x="180.34" y="215.9"/>
+<wire x1="162.56" y1="218.44" x2="162.56" y2="215.9" width="0.1524" layer="91"/>
+<wire x1="154.94" y1="220.98" x2="154.94" y2="218.44" width="0.1524" layer="91"/>
+<wire x1="154.94" y1="218.44" x2="162.56" y2="218.44" width="0.1524" layer="91"/>
+<junction x="162.56" y="218.44"/>
 <pinref part="R18" gate="G$1" pin="2"/>
-<wire x1="172.72" y1="215.9" x2="172.72" y2="213.36" width="0.1524" layer="91"/>
-<junction x="172.72" y="215.9"/>
+<wire x1="154.94" y1="218.44" x2="154.94" y2="215.9" width="0.1524" layer="91"/>
+<junction x="154.94" y="218.44"/>
 <pinref part="TP9" gate="G$1" pin="TP"/>
-<wire x1="180.34" y1="215.9" x2="187.96" y2="215.9" width="0.1524" layer="91"/>
+<wire x1="162.56" y1="218.44" x2="170.18" y2="218.44" width="0.1524" layer="91"/>
 </segment>
 </net>

Commit message: included qwertyembedded work
Connections:
- new net RESET: TP14.TP, U$4./RESET
- new net SWCLK: TP15.TP, U$4.PA30/I10/SECOM1.2/SWCLK
- new net SWDIO: TP16.TP, U$4.PA31/I11/SECOM1.3/SWDIO
- net USB_N: now also TP12.TP
- net USB_P: now also TP13.TP
Other:
- moved on the sheet: TP12, TP13, TP14, TP15, TP16
Changed lines of the file:
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@@
 <attribute name="TP_SIGNAL_NAME" x="11.43" y="179.07" size="1.778" layer="97"/>
 </instance>
-<instance part="TP12" gate="G$1" x="15.24" y="180.34" smashed="yes">
-<attribute name="NAME" x="13.97" y="181.61" size="1.778" layer="95"/>
-<attribute name="TP_SIGNAL_NAME" x="16.51" y="179.07" size="1.778" layer="97"/>
+<instance part="TP12" gate="G$1" x="139.7" y="35.56" smashed="yes">
+<attribute name="NAME" x="138.43" y="36.83" size="1.778" layer="95"/>
+<attribute name="TP_SIGNAL_NAME" x="140.97" y="34.29" size="1.778" layer="97"/>
 </instance>
-<instance part="TP13" gate="G$1" x="20.32" y="180.34" smashed="yes">
-<attribute name="NAME" x="19.05" y="181.61" size="1.778" layer="95"/>
-<attribute name="TP_SIGNAL_NAME" x="21.59" y="179.07" size="1.778" layer="97"/>
+<instance part="TP13" gate="G$1" x="144.78" y="33.02" smashed="yes">
+<attribute name="NAME" x="143.51" y="34.29" size="1.778" layer="95"/>
+<attribute name="TP_SIGNAL_NAME" x="146.05" y="31.75" size="1.778" layer="97"/>
 </instance>
-<instance part="TP14" gate="G$1" x="25.4" y="180.34" smashed="yes">
-<attribute name="NAME" x="24.13" y="181.61" size="1.778" layer="95"/>
-<attribute name="TP_SIGNAL_NAME" x="26.67" y="179.07" size="1.778" layer="97"/>
+<instance part="TP14" gate="G$1" x="43.18" y="101.6" smashed="yes">
+<attribute name="NAME" x="41.91" y="102.87" size="1.778" layer="95"/>
+<attribute name="TP_SIGNAL_NAME" x="44.45" y="100.33" size="1.778" layer="97"/>
 </instance>
-<instance part="TP15" gate="G$1" x="30.48" y="180.34" smashed="yes">
-<attribute name="NAME" x="29.21" y="181.61" size="1.778" layer="95"/>
-<attribute name="TP_SIGNAL_NAME" x="31.75" y="179.07" size="1.778" layer="97"/>
+<instance part="TP15" gate="G$1" x="132.08" y="25.4" smashed="yes">
+<attribute name="NAME" x="130.81" y="26.67" size="1.778" layer="95"/>
+<attribute name="TP_SIGNAL_NAME" x="133.35" y="24.13" size="1.778" layer="97"/>
 </instance>
-<instance part="TP16" gate="G$1" x="35.56" y="180.34" smashed="yes">
-<attribute name="NAME" x="34.29" y="181.61" size="1.778" layer="95"/>
-<attribute name="TP_SIGNAL_NAME" x="36.83" y="179.07" size="1.778" layer="97"/>
+<instance part="TP16" gate="G$1" x="137.16" y="22.86" smashed="yes">
+<attribute name="NAME" x="135.89" y="24.13" size="1.778" layer="95"/>
+<attribute name="TP_SIGNAL_NAME" x="138.43" y="21.59" size="1.778" layer="97"/>
 </instance>
 </instances>
@@
 <label x="49.53" y="-123.19" size="1.778" layer="95"/>
 </segment>
+<segment>
+<pinref part="U$4" gate="G$1" pin="PA30/I10/SECOM1.2/SWCLK"/>
+<pinref part="TP15" gate="G$1" pin="TP"/>
+<wire x1="119.38" y1="22.86" x2="132.08" y2="22.86" width="0.1524" layer="91"/>
+<label x="121.92" y="22.86" size="1.778" layer="95"/>
+</segment>
 </net>
 <net name="SWDIO" class="0">
@@
 <wire x1="59.69" y1="-125.73" x2="41.91" y2="-125.73" width="0.1524" layer="91"/>
 <label x="49.53" y="-125.73" size="1.778" layer="95"/>
+</segment>
+<segment>
+<pinref part="U$4" gate="G$1" pin="PA31/I11/SECOM1.3/SWDIO"/>
+<pinref part="TP16" gate="G$1" pin="TP"/>
+<wire x1="119.38" y1="20.32" x2="137.16" y2="20.32" width="0.1524" layer="91"/>
+<label x="121.92" y="20.32" size="1.778" layer="95"/>
 </segment>
 </net>
@@
 <label x="127" y="33.02" size="1.778" layer="95"/>
 <pinref part="U$4" gate="G$1" pin="PA24/I12/SERCOM3+5.2/D-"/>
+<pinref part="TP12" gate="G$1" pin="TP"/>
+<wire x1="137.16" y1="33.02" x2="139.7" y2="33.02" width="0.1524" layer="91"/>
 </segment>
 </net>
@@
 <label x="127" y="30.48" size="1.778" layer="95"/>
 <pinref part="U$4" gate="G$1" pin="PA25/I13/SERCOM3+5.3/D+"/>
-</segment>
-</net>
+<pinref part="TP13" gate="G$1" pin="TP"/>
+<wire x1="137.16" y1="30.48" x2="144.78" y2="30.48" width="0.1524" layer="91"/>
+</segment>
+</net>
+<net name="RESET" class="0">
+<segment>
+<pinref part="U$4" gate="G$1" pin="/RESET"/>
+<pinref part="TP14" gate="G$1" pin="TP"/>
+<wire x1="50.8" y1="99.06" x2="43.18" y2="99.06" width="0.1524" layer="91"/>
+<label x="45.72" y="99.06" size="1.778" layer="95"/>
+</segment>
+</net>

Commit message: ratsnestnothing to do
Parts:
- removed C28: 1uF, microbuilder:CAP_CERAMIC0603_NO
- removed U$4: ATSAMD21J18A-AUT, ATSam21:ATSAMD21J18A-AUT
- added DIODES: TDP3E001DRLR-SOT-23-5SOT-23-5, USBC:TDP3E001DRLR-SOT-23-5SOT-23-5
- added R19: 0, SparkFun-Resistors:5.62KOHM-0603-1/10W-1%
- added TP17: TPB1,27, testpad:TPB1,27
- U1: value TDP3E001DRLR-SOT-23-5SOT-23-5 -> ATSAMD21J18A-AUT; device USBC:TDP3E001DRLR-SOT-23-5SOT-23-5 -> ATSam21:ATSAMD21J18A-AUT
Connections:
- removed net !RESET: SW1.P, SW1.P1
- removed net N$53: U6.T2OUT
- removed net VDDCORE2: C28.1
- new net N$1: U$5.P3, U6.R1IN
- new net PB31: U$32.3V3@1, U1.PB31
- new net UART_RX: U$32.RXD0/GPIO15, U1.PA09/I2C/I9/AIN17/SERCOM0+2.1/I2SMC, U6.R1OUT
- new net UART_TX: U$32.TXD0/GPIO14, U1.PA08/I2C/AIN16/SERCOM0+2.0/I2SD1, U6.T1IN
- new net VCC: R19.2
- net 3V3: now also R19.1, U1.VDDA, U1.VDDIN, U1.VDDIO, U6.VCC
- net GND: now also DIODES.3, U$5.P5, U1.GND, U1.GNDA, U6.GND; no longer C28.2, U1.3
- net KEYCOLUMN0: now also U1.PA10/I10/AIN18/SERCOM0+2.2/I2SCK
- net KEYCOLUMN1: now also U1.PA11/I11/AIN19/SERCOM0+2.3/I2SF0
- net KEYCOLUMN10: now also U1.PA20/I4/SERCOM3+5.2/I2SSC
- net KEYCOLUMN11: now also U1.PA21/I5/SERCOM3/5.3/I2SFS0
- net KEYCOLUMN12: now also U1.PA15/I15/SERCOM3+4.3
- net KEYCOLUMN13: now also U1.PA22/I2C/I6/SERCOM3+5.0
- net KEYCOLUMN14: now also U1.PA27/I15
- net KEYCOLUMN15: now also U1.PA28/I8
- net KEYCOLUMN2: now also U1.PA12/I12/I2C/SERCOM2+4.0
- net KEYCOLUMN3: now also U1.PA13/I13/I2C/SERCOM2+4.1
- net KEYCOLUMN4: now also U1.PA07/AIN7/SERCOM0.3/I2SD0
- net KEYCOLUMN5: now also U1.PA14/I14/SERCOM2+4.2
- net KEYCOLUMN6: now also U1.PA16/I2C/I0/SERCOM1+3.0
- net KEYCOLUMN7: now also U1.PA17/I2C/I1/SERCOM1+3.1
- net KEYCOLUMN8: now also U1.PA18/I2/SERCOM1+3.2
- net KEYCOLUMN9: now also U1.PA19/I3/SERCOM1+3.3/I2SD0
- net KEYROW0: now also U1.PA02/EINT2/AIN0/Y0/VOUT
- net KEYROW1: now also U1.PA03/EINT3/VREFA/AIN1
- net KEYROW2: now also U1.PA04/EINT4/VREFB/AIN4/SERCOM0.0
- net KEYROW3: now also U1.PA05/EINT5/AIN5/SERCOM0.1
- net KEYROW4: now also U1.PA06/EINT6/AIN6/SSERCOM0.2
- net LCD0: now also U1.PB00; no longer U$4.PB00
- net LCD1: now also U1.PB01; no longer U$4.PB01
- net LCD10: now also U1.PB10; no longer U$4.PB10
- net LCD11: now also U1.PB11; no longer U$4.PB11
- net LCD12: now also U1.PB12; no longer U$4.PB12
- net LCD13: now also U1.PB13; no longer U$4.PB13
- net LCD14: now also U1.PB14; no longer U$4.PB14
- net LCD15: now also U1.PB15; no longer U$4.PB15
- net LCD2: now also U1.PB02; no longer U$4.PB02
- net LCD3: now also U1.PB03; no longer U$4.PB03
- net LCD4: now also U1.PB04; no longer U$4.PB04
- net LCD5: now also U1.PB05; no longer U$4.PB05
- net LCD6: now also U1.PB06; no longer U$4.PB06
- net LCD7: now also U1.PB07; no longer U$4.PB07
- net LCD8: now also U1.PB08; no longer U$4.PB08
- net LCD9: now also U1.PB09; no longer U$4.PB09
- net LCD_CS: now also U1.PB22; no longer U$4.PB22
- net LCD_D/C: now also U1.PB23; no longer U$4.PB23
- net LCD_RD: now also U1.PB16; no longer U$4.PB16
- net LCD_RESET: now also U1.PB30; no longer U$4.PB30
- net LCD_W/R: now also U1.PB17; no longer U$4.PB17
- net N$52: now also U$5.P2
- net N$54: now also U1.PA00/EINT0/SERCOM1.0
- net N$55: now also U1.PA01/EINT1/SERCOM1.1
- net PWM: now also TP17.TP
- net RESET: now also SW1.P, SW1.P1, U1./RESET; no longer U$4./RESET
- net SWCLK: now also U1.PA30/I10/SECOM1.2/SWCLK; no longer U$4.PA30/I10/SECOM1.2/SWCLK
- net SWDIO: now also U1.PA31/I11/SECOM1.3/SWDIO; no longer U$4.PA31/I11/SECOM1.3/SWDIO
- net USB_N: now also DIODES.IO1, U1.PA24/I12/SERCOM3+5.2/D-; no longer U$4.PA24/I12/SERCOM3+5.2/D-, U1.IO1
- net USB_P: now also DIODES.IO2, U1.PA25/I13/SERCOM3+5.3/D+; no longer U$4.PA25/I13/SERCOM3+5.3/D+, U1.IO2
- net VBUS: now also DIODES.5; no longer U1.5
Other:
- note removed: "N/C"
- note removed: "RESET"
- note removed: "TXLED"
- note removed: "USBHOSTEN"
- moved on the sheet: C22, C23, C24, C26, C27, IC1, IC2, IC3, SW1, TP12, TP13, TP14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
