File: Electronics/DumbBadgeFusion.brd (EAGLE design)
At the start: 163.5 x 113 mm, 148 parts, among them IC1 74245MTC, IC2 74245MTC, IC3 74245MTC, SW1 SPST_TACT-KMR2, T1 MMUN2133LT1G, U1 TDP3E001DRLR-SOT-23-5SOT-23-5, U2 TPS61090RSAR, U3 MCP73871, U4 FAN5333BSX, U6 MAX3232, X4 32.768

Commit message: included qwertyembedded work
Connections:
- new net RESET: TP14.TP, U$4.52
- new net SWCLK: TP15.TP, U$4.57
- new net SWDIO: TP16.TP, U$4.58
- net USB_N: now also TP12.TP
- net USB_P: now also TP13.TP
Other:
- board text added: "USB+"
- board text added: "USB-"
- board text added: "reset"
- board text added: "swclk"
- board text added: "swdio"
Changed lines of the file:
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@@
 <text x="17.78" y="55.88" size="1.27" layer="22" font="vector" ratio="14" rot="MR0" align="center">GND</text>
 <text x="17.78" y="62.23" size="1.27" layer="22" font="vector" ratio="14" rot="MR0" align="center">V+</text>
+<text x="103.378" y="51.308" size="0.6096" layer="22" font="vector" ratio="14" rot="MR0" align="center">swclk</text>
+<text x="105.918" y="51.308" size="0.6096" layer="22" font="vector" ratio="14" rot="MR0" align="center">swdio</text>
+<text x="100.838" y="51.308" size="0.6096" layer="22" font="vector" ratio="14" rot="MR0" align="center">reset</text>
+<text x="98.298" y="51.308" size="0.6096" layer="22" font="vector" ratio="14" rot="MR0" align="center">USB+</text>
+<text x="95.758" y="51.308" size="0.6096" layer="22" font="vector" ratio="14" rot="MR0" align="center">USB-</text>
 </plain>
 <attributes>
@@
 <wire x1="155.575" y1="98.964" x2="155.623" y2="99.012" width="0.3048" layer="16"/>
 <contactref element="U$4" pad="46"/>
+<contactref element="TP13" pad="TP"/>
 <wire x1="153.3953" y1="99.6696" x2="137.6140375" y2="80.90505" width="0" layer="19" extent="16-16"/>
+<wire x1="98.298" y1="52.324" x2="137.6140375" y2="80.90505" width="0" layer="19" extent="16-16"/>
 </signal>
 <signal name="USB_N">
@@
 <wire x1="158.933" y1="99.512" x2="157.63" y2="99.512" width="0.3048" layer="16"/>
 <contactref element="U$4" pad="45"/>
+<contactref element="TP12" pad="TP"/>
 <wire x1="153.3953" y1="100.6196" x2="137.260484375" y2="80.551496875" width="0" layer="19" extent="16-16"/>
+<wire x1="95.758" y1="52.324" x2="137.260484375" y2="80.551496875" width="0" layer="19" extent="16-16"/>
 </signal>
 <signal name="LCD0">
@@
 <via x="37.338" y="54.483" extent="1-16" drill="0.2"/>
 <wire x1="34.912325" y1="49.8364" x2="37.2856" y2="52.209675" width="0.254" layer="1"/>
-<wire x1="30.48" y1="52.2572625" x2="30.57363125" y2="52.16363125" width="0.254" layer="1"/>
-<wire x1="30.57363125" y1="52.16363125" x2="32.9008625" y2="49.8364" width="0.254" layer="1"/>
-<wire x1="32.9008625" y1="49.8364" x2="34.912325" y2="49.8364" width="0.254" layer="1"/>
+<wire x1="32.9008625" y1="49.8364" x2="33.02" y2="49.8364" width="0.254" layer="1"/>
+<wire x1="33.02" y1="49.8364" x2="34.912325" y2="49.8364" width="0.254" layer="1"/>
 <wire x1="37.338" y1="52.324" x2="37.2856" y2="52.2716" width="0.254" layer="1"/>
 <wire x1="37.338" y1="52.324" x2="37.338" y2="54.483" width="0.254" layer="1"/>
@@
 <wire x1="26.797" y1="109.982" x2="28.067" y2="108.712" width="0.4064" layer="1"/>
 <wire x1="28.067" y1="108.712" x2="28.067" y2="70.104" width="0.4064" layer="1"/>
-<wire x1="30.57363125" y1="52.16363125" x2="30.1592625" y2="52.578" width="0.254" layer="1"/>
-<wire x1="30.1592625" y1="52.578" x2="18.77794375" y2="52.578" width="0.254" layer="1"/>
+<wire x1="33.02" y1="49.8364" x2="23.4426" y2="49.8364" width="0.254" layer="1"/>
+<wire x1="20.701" y1="52.578" x2="18.77794375" y2="52.578" width="0.254" layer="1"/>
+<wire x1="23.4426" y1="49.8364" x2="20.701" y2="52.578" width="0.254" layer="1"/>
+</signal>
+<signal name="SWCLK">
+<contactref element="U$4" pad="57"/>
+<contactref element="TP15" pad="TP"/>
+<wire x1="103.378" y1="52.324" x2="143.9072875" y2="78.78373125" width="0" layer="19" extent="16-16"/>
+</signal>
+<signal name="SWDIO">
+<contactref element="U$4" pad="58"/>
+<contactref element="TP16" pad="TP"/>
+<wire x1="105.918" y1="52.324" x2="144.260840625" y2="78.430178125" width="0" layer="19" extent="16-16"/>
+</signal>
+<signal name="RESET">
+<contactref element="U$4" pad="52"/>
+<contactref element="TP14" pad="TP"/>
+<wire x1="100.838" y1="52.324" x2="142.13951875" y2="80.551496875" width="0" layer="19" extent="16-16"/>
 </signal>
 </signals>
