File: Extensions/EmbiggenedKeyboard/EmbiggenedKeyboard.brd (EAGLE design)
At the start: 324 x 112 mm, 75 parts

Commit message: thing
Parts:
- removed ?/, LEFTSHIFT, PIPE, RETURN, RETURN2, RIGHTSHIFT, SETUP, SPACE1: KEYSWITCH-PLAIN-MX-1U, Keyboard:MX-1U
- removed J1: (no value), SparkFun-Connectors:1X17
- removed J2, J3: (no value), SparkFun-Connectors:1X15
- added K-1, K-2, K-5, K_0, K_3, K_4, K_6, K_7, K_8, K_9, K_<, K_>, K_?, K_A, K_B, K_BACK, K_BREAK, K_C, K_CAPS, K_D, K_DEL, K_DOWN, K_E, K_ESC, K_F, K_G, K_H, K_I, K_J, K_K, K_L, K_LEFT, K_LEFTALT, K_LEFTMETA, K_LINE, K_M, K_N, K_NOSCL, K_O, K_P, K_PIPE, K_PLUS, K_Q, K_QUOTE, K_R, K_RIGHT, K_RIGHTALT, K_RIGHTMETA, K_S, K_SEMI, K_T, K_TAB, K_TILDE, K_U, K_UP, K_USCORE, K_V, K_W, K_X, K_Y, K_Z, K_{, K_}: 1U_PAD, SiliconeSwitches:SILICONE_SWITCH
- added K_CONTROL, K_LSHIFT, K_RSHIFT, K_SETUP: 2U_PAD, SiliconeSwitches:SILICONE_SWITCH_2U
- added K_RETURN: RETURN_PAD, SiliconeSwitches:SILICONE_RETURN
- added K_SPACE: SPACE_PAD, SiliconeSwitches:SILICONE_SPACE
- added SHIFT, SHIFT2, SPACE, \|: KEYSWITCH-PLAIN-MX-1U, Keyboard:MX-1U
- moved SPACE2 142.1 mm to (290.5, -57.1)
- moved LINE 133.4 mm to (295.3, -85.7)
- moved SPACE3 129.9 mm to (157.2, -104.8)
- moved ALT 114.6 mm to (61.9, -104.8)
- moved META 113.4 mm to (42.9, -104.8)
- moved TAB 113.4 mm to (28.6, -47.6)
- moved B 113.1 mm to (152.4, -85.7)
- moved C 113.1 mm to (114.3, -85.7)
- moved COMMA 113.1 mm to (209.6, -85.7)
- moved M 113.1 mm to (190.5, -85.7)
- moved N 113.1 mm to (171.4, -85.7)
- moved PERIOD 113.1 mm to (228.6, -85.7)
- moved V 113.1 mm to (133.3, -85.7)
- moved X 113.1 mm to (95.2, -85.7)
- moved Z 113.1 mm to (76.2, -85.7)
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Connections:
- net KEYCOLUM0: now also K_7.P$2, K_<.P$2, K_ESC.P$2, K_G.P$2, K_J.P$2, K_NOSCL.P$2, K_RIGHTALT.P$2, K_SETUP.P$2, K_TAB.P$2, K_U.P$2; no longer 7.MX1, ALT2.MX1, COMMA.MX1, ESC.MX1, G.MX1, J.MX1, J1.7, J2.15, NO.MX1, SETUP.MX1, TAB.MX1, U.MX1
- net KEYCOLUM1: now also K-1.P$2, K_8.P$2, K_CAPS.P$2, K_H.P$2, K_I.P$2, K_K.P$2, K_LSHIFT.P$2, K_Q.P$2, K_RIGHTMETA.P$2; no longer 1.MX1, 8.MX1, CAPS.MX1, H.MX1, I.MX1, J1.6, J2.14, K.MX1, LEFTSHIFT.MX1, META2.MX1, Q.MX1
- net KEYCOLUM2: now also K-2.P$2, K_0.P$2, K_9.P$2, K_>.P$2, K_CONTROL.P$2, K_L.P$2, K_LEFTMETA.P$2, K_O.P$2, K_W.P$2, K_Z.P$2; no longer 0.MX1, 2.MX1, 9.MX1, CTRL.MX1, J1.5, J2.13, L.MX1, META.MX1, O.MX1, PERIOD.MX1, W.MX1, Z.MX1
- net KEYCOLUM3: now also K_3.P$2, K_?.P$2, K_A.P$2, K_E.P$2, K_LEFT.P$2, K_LEFTALT.P$2, K_P.P$2, K_SEMI.P$2, K_USCORE.P$2, K_X.P$2; no longer 3.MX1, ?/.MX1, A.MX1, ALT.MX1, E.MX1, J1.4, J2.12, KP_DASH.MX1, LEFT.MX1, P.MX1, SEMI.MX1, X.MX1
- net KEYCOLUM4: now also K_4.P$2, K_C.P$2, K_DOWN.P$2, K_PLUS.P$2, K_QUOTE.P$2, K_R.P$2, K_RSHIFT.P$2, K_S.P$2, K_SPACE.P$2, K_{.P$2; no longer 4.MX1, C.MX1, DOWN.MX1, EQUAL.MX1, J1.3, J2.11, LBRACKET.MX1, QUOTE.MX1, R.MX1, RIGHTSHIFT.MX1, S.MX1, SPACE1.MX1, SPACE2.MX1, SPACE3.MX1
- net KEYCOLUM5: now also K-5.P$2, K_D.P$2, K_N.P$2, K_PIPE.P$2, K_RETURN.P$2, K_T.P$2, K_TILDE.P$2, K_UP.P$2, K_V.P$2, K_}.P$2; no longer 5.MX1, D.MX1, GRAVE.MX1, J1.2, J2.10, N.MX1, PIPE.MX1, RBRACKET.MX1, RETURN.MX1, RETURN2.MX1, T.MX1, UP.MX1, V.MX1
- net KEYCOLUM6: now also K_6.P$2, K_B.P$2, K_BACK.P$2, K_BREAK.P$2, K_DEL.P$2, K_F.P$2, K_LINE.P$2, K_M.P$2, K_RIGHT.P$2, K_Y.P$2; no longer 6.MX1, B.MX1, BACK.MX1, BRK.MX1, DEL.MX1, F.MX1, J1.1, J2.9, LINE.MX2, M.MX1, RIGHT.MX1, Y.MX1
- net KEYROW0: now also K-1.P$1, K-2.P$1, K-5.P$1, K_3.P$1, K_4.P$1, K_6.P$1, K_ESC.P$1; no longer 1.MX2, 2.MX2, 3.MX2, 4.MX2, 5.MX2, 6.MX2, ESC.MX2, J1.17, J3.15
- net KEYROW1: now also K_E.P$1, K_Q.P$1, K_R.P$1, K_SETUP.P$1, K_T.P$1, K_W.P$1, K_Y.P$1; no longer E.MX2, J1.16, J3.14, Q.MX2, R.MX2, SETUP.MX2, T.MX2, W.MX2, Y.MX2
- net KEYROW2: now also K_A.P$1, K_CAPS.P$1, K_CONTROL.P$1, K_D.P$1, K_F.P$1, K_S.P$1, K_TAB.P$1; no longer A.MX2, CAPS.MX2, CTRL.MX2, D.MX2, F.MX2, J1.15, J3.13, S.MX2, TAB.MX2
- net KEYROW3: now also K_B.P$1, K_C.P$1, K_LSHIFT.P$1, K_NOSCL.P$1, K_V.P$1, K_X.P$1, K_Z.P$1; no longer B.MX2, C.MX2, J1.14, J3.12, LEFTSHIFT.MX2, NO.MX2, V.MX2, X.MX2, Z.MX2
- net KEYROW4: now also K_LEFTALT.P$1, K_LEFTMETA.P$1, K_M.P$1, K_N.P$1, K_RIGHTALT.P$1, K_RIGHTMETA.P$1, K_SPACE.P$1; no longer ALT.MX2, ALT2.MX2, J1.13, J3.11, M.MX2, META.MX2, META2.MX2, N.MX2, SPACE1.MX2, SPACE2.MX2, SPACE3.MX2
- net KEYROW5: now also K_7.P$1, K_8.P$1, K_9.P$1, K_DOWN.P$1, K_LEFT.P$1, K_RIGHT.P$1, K_UP.P$1; no longer 7.MX2, 8.MX2, 9.MX2, DOWN.MX2, J1.12, J3.10, LEFT.MX2, RIGHT.MX2, UP.MX2
- net KEYROW6: now also K_0.P$1, K_BACK.P$1, K_I.P$1, K_PLUS.P$1, K_TILDE.P$1, K_U.P$1, K_USCORE.P$1; no longer 0.MX2, BACK.MX2, EQUAL.MX2, GRAVE.MX2, I.MX2, J1.11, J3.9, KP_DASH.MX2, U.MX2
- net KEYROW7: now also K_BREAK.P$1, K_G.P$1, K_H.P$1, K_O.P$1, K_P.P$1, K_{.P$1, K_}.P$1; no longer BRK.MX2, G.MX2, H.MX2, J1.10, J3.8, LBRACKET.MX2, O.MX2, P.MX2, RBRACKET.MX2
- net KEYROW8: now also K_DEL.P$1, K_J.P$1, K_K.P$1, K_L.P$1, K_QUOTE.P$1, K_RETURN.P$1, K_SEMI.P$1; no longer DEL.MX2, J.MX2, J1.9, J3.7, K.MX2, L.MX2, QUOTE.MX2, RETURN.MX2, RETURN2.MX2, SEMI.MX2
- net KEYROW9: now also K_<.P$1, K_>.P$1, K_?.P$1, K_LINE.P$1, K_PIPE.P$1, K_RSHIFT.P$1; no longer ?/.MX2, COMMA.MX2, J1.8, J3.6, LINE.MX1, PERIOD.MX2, PIPE.MX2, RIGHTSHIFT.MX2
Routing:
- net KEYCOLUM5: track 630.9 -> 0.00 mm, vias 1 -> 0
- net KEYCOLUM6: track 598.5 -> 0.00 mm, vias 2 -> 0
- net KEYCOLUM4: track 553.9 -> 0.00 mm, vias 2 -> 0
- net KEYCOLUM1: track 519.6 -> 0.00 mm, vias 2 -> 0
- net KEYCOLUM0: track 496.4 -> 0.00 mm, vias 4 -> 0
- net KEYROW4: track 480.6 -> 0.00 mm, vias 5 -> 0
- net KEYCOLUM3: track 478.5 -> 0.00 mm
- net KEYCOLUM2: track 457.0 -> 0.00 mm
- net KEYROW8: track 406.1 -> 0.00 mm, vias 3 -> 0
- net KEYROW3: track 400.2 -> 0.00 mm, vias 1 -> 0
- net KEYROW9: track 398.5 -> 0.00 mm, vias 3 -> 0
- net KEYROW7: track 392.1 -> 0.00 mm, vias 3 -> 0
- net KEYROW6: track 353.2 -> 0.00 mm, vias 2 -> 0
- net KEYROW5: track 332.1 -> 0.00 mm, vias 2 -> 0
- net KEYROW1: track 325.8 -> 0.00 mm, vias 2 -> 0
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- removed copper zone on layer 16, net GND
- removed copper zone on layer 1, net VCC
Other:
- board text removed: "0"
- board text removed: "1"
- board text removed: "2"
- board text removed: "3"
- board text removed: "4"
- board text removed: "5"
- board text removed: "6"
- board text removed: "69% BARF BOARD"
- board text removed: "7"
- board text removed: "8"
- board text removed: "9"
- board text removed: "COLUMN"
- board text removed: "ROW"
