File: Extensions/EmbiggenedKeyboard/EmbiggenedKeyboard.sch (EAGLE design)
At the start: 137 parts

Commit message: This doesn't fix the cursor problem, but it's better
redid everything so pixel 0,0 is in the upper left
Parts:
- removed K-1, K-2, K-5, K_0, K_3, K_4, K_6, K_7, K_8, K_9, K_<, K_>, K_?, K_A, K_B, K_BACK, K_BREAK, K_C, K_CAPS, K_D, K_DEL, K_DOWN, K_E, K_ESC, K_F, K_G, K_H, K_I, K_J, K_K, K_L, K_LEFT, K_LEFTALT, K_LEFTMETA, K_LINE, K_M, K_N, K_NOSCL, K_O, K_P, K_PIPE, K_PLUS, K_Q, K_QUOTE, K_R, K_RIGHT, K_RIGHTALT, K_RIGHTMETA, K_S, K_SEMI, K_T, K_TAB, K_TILDE, K_U, K_UP, K_USCORE, K_V, K_W, K_X, K_Y, K_Z, K_{, K_}: 1U_PAD, SiliconeSwitches:1U_PAD
- removed K_CONTROL, K_LSHIFT, K_RSHIFT, K_SETUP: 2U_PAD, SiliconeSwitches:2U_PAD
- removed K_RETURN: RETURN_PAD, SiliconeSwitches:RETURN_PAD
- removed K_SPACE: SPACE_PAD, SiliconeSwitches:SPACE_PAD
- removed SHIFT, SHIFT2, SPACE, \|: KEYSWITCH-PLAIN-MX-1U, Keyboard:KEYSWITCH-PLAIN-MX-1U
- added ?/, LEFTSHIFT, PIPE, RETURN, RETURN2, RIGHTSHIFT, SETUP, SPACE1: KEYSWITCH-PLAIN-MX-1U, Keyboard:KEYSWITCH-PLAIN-MX-1U
- added J1: (no value), SparkFun-Connectors:CONN_17
- added J2, J3: (no value), SparkFun-Connectors:CONN_15
Connections:
- net KEYCOLUM0: now also 7.P0, ALT2.P0, COMMA.P0, ESC.P0, G.P0, J.P0, J1.7, J2.15, NO.P0, SETUP.P0, TAB.P0, U.P0; no longer K_7.P$2, K_<.P$2, K_ESC.P$2, K_G.P$2, K_J.P$2, K_NOSCL.P$2, K_RIGHTALT.P$2, K_SETUP.P$2, K_TAB.P$2, K_U.P$2
- net KEYCOLUM1: now also 1.P0, 8.P0, CAPS.P0, H.P0, I.P0, J1.6, J2.14, K.P0, LEFTSHIFT.P0, META2.P0, Q.P0; no longer K-1.P$2, K_8.P$2, K_CAPS.P$2, K_H.P$2, K_I.P$2, K_K.P$2, K_LSHIFT.P$2, K_Q.P$2, K_RIGHTMETA.P$2
- net KEYCOLUM2: now also 0.P0, 2.P0, 9.P0, CTRL.P0, J1.5, J2.13, L.P0, META.P0, O.P0, PERIOD.P0, W.P0, Z.P0; no longer K-2.P$2, K_0.P$2, K_9.P$2, K_>.P$2, K_CONTROL.P$2, K_L.P$2, K_LEFTMETA.P$2, K_O.P$2, K_W.P$2, K_Z.P$2
- net KEYCOLUM3: now also 3.P0, ?/.P0, A.P0, ALT.P0, E.P0, J1.4, J2.12, KP_DASH.P0, LEFT.P0, P.P0, SEMI.P0, X.P0; no longer K_3.P$2, K_?.P$2, K_A.P$2, K_E.P$2, K_LEFT.P$2, K_LEFTALT.P$2, K_P.P$2, K_SEMI.P$2, K_USCORE.P$2, K_X.P$2
- net KEYCOLUM4: now also 4.P0, C.P0, DOWN.P0, EQUAL.P0, J1.3, J2.11, LBRACKET.P0, QUOTE.P0, R.P0, RIGHTSHIFT.P0, S.P0, SPACE1.P0, SPACE2.P0, SPACE3.P0; no longer K_4.P$2, K_C.P$2, K_DOWN.P$2, K_PLUS.P$2, K_QUOTE.P$2, K_R.P$2, K_RSHIFT.P$2, K_S.P$2, K_SPACE.P$2, K_{.P$2
- net KEYCOLUM5: now also 5.P0, D.P0, GRAVE.P0, J1.2, J2.10, N.P0, PIPE.P0, RBRACKET.P0, RETURN.P0, RETURN2.P0, T.P0, UP.P0, V.P0; no longer K-5.P$2, K_D.P$2, K_N.P$2, K_PIPE.P$2, K_RETURN.P$2, K_T.P$2, K_TILDE.P$2, K_UP.P$2, K_V.P$2, K_}.P$2
- net KEYCOLUM6: now also 6.P0, B.P0, BACK.P0, BRK.P0, DEL.P0, F.P0, J1.1, J2.9, LINE.P1, M.P0, RIGHT.P0, Y.P0; no longer K_6.P$2, K_B.P$2, K_BACK.P$2, K_BREAK.P$2, K_DEL.P$2, K_F.P$2, K_LINE.P$2, K_M.P$2, K_RIGHT.P$2, K_Y.P$2
- net KEYROW0: now also 1.P1, 2.P1, 3.P1, 4.P1, 5.P1, 6.P1, ESC.P1, J1.17, J3.15; no longer K-1.P$1, K-2.P$1, K-5.P$1, K_3.P$1, K_4.P$1, K_6.P$1, K_ESC.P$1
- net KEYROW1: now also E.P1, J1.16, J3.14, Q.P1, R.P1, SETUP.P1, T.P1, W.P1, Y.P1; no longer K_E.P$1, K_Q.P$1, K_R.P$1, K_SETUP.P$1, K_T.P$1, K_W.P$1, K_Y.P$1
- net KEYROW2: now also A.P1, CAPS.P1, CTRL.P1, D.P1, F.P1, J1.15, J3.13, S.P1, TAB.P1; no longer K_A.P$1, K_CAPS.P$1, K_CONTROL.P$1, K_D.P$1, K_F.P$1, K_S.P$1, K_TAB.P$1
- net KEYROW3: now also B.P1, C.P1, J1.14, J3.12, LEFTSHIFT.P1, NO.P1, V.P1, X.P1, Z.P1; no longer K_B.P$1, K_C.P$1, K_LSHIFT.P$1, K_NOSCL.P$1, K_V.P$1, K_X.P$1, K_Z.P$1
- net KEYROW4: now also ALT.P1, ALT2.P1, J1.13, J3.11, M.P1, META.P1, META2.P1, N.P1, SPACE1.P1, SPACE2.P1, SPACE3.P1; no longer K_LEFTALT.P$1, K_LEFTMETA.P$1, K_M.P$1, K_N.P$1, K_RIGHTALT.P$1, K_RIGHTMETA.P$1, K_SPACE.P$1
- net KEYROW5: now also 7.P1, 8.P1, 9.P1, DOWN.P1, J1.12, J3.10, LEFT.P1, RIGHT.P1, UP.P1; no longer K_7.P$1, K_8.P$1, K_9.P$1, K_DOWN.P$1, K_LEFT.P$1, K_RIGHT.P$1, K_UP.P$1
- net KEYROW6: now also 0.P1, BACK.P1, EQUAL.P1, GRAVE.P1, I.P1, J1.11, J3.9, KP_DASH.P1, U.P1; no longer K_0.P$1, K_BACK.P$1, K_I.P$1, K_PLUS.P$1, K_TILDE.P$1, K_U.P$1, K_USCORE.P$1
- net KEYROW7: now also BRK.P1, G.P1, H.P1, J1.10, J3.8, LBRACKET.P1, O.P1, P.P1, RBRACKET.P1; no longer K_BREAK.P$1, K_G.P$1, K_H.P$1, K_O.P$1, K_P.P$1, K_{.P$1, K_}.P$1
- net KEYROW8: now also DEL.P1, J.P1, J1.9, J3.7, K.P1, L.P1, QUOTE.P1, RETURN.P1, RETURN2.P1, SEMI.P1; no longer K_DEL.P$1, K_J.P$1, K_K.P$1, K_L.P$1, K_QUOTE.P$1, K_RETURN.P$1, K_SEMI.P$1
- net KEYROW9: now also ?/.P1, COMMA.P1, J1.8, J3.6, LINE.P0, PERIOD.P1, PIPE.P1, RIGHTSHIFT.P1; no longer K_<.P$1, K_>.P$1, K_?.P$1, K_LINE.P$1, K_PIPE.P$1, K_RSHIFT.P$1
Other:
- moved on the sheet: 0, 1, 2, 3, 4, 5, 6, 7, 8, 9, A, ALT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

Commit message: thing
Parts:
- removed ?/, LEFTSHIFT, PIPE, RETURN, RETURN2, RIGHTSHIFT, SETUP, SPACE1: KEYSWITCH-PLAIN-MX-1U, Keyboard:KEYSWITCH-PLAIN-MX-1U
- removed J1: (no value), SparkFun-Connectors:CONN_17
- removed J2, J3: (no value), SparkFun-Connectors:CONN_15
- added K-1, K-2, K-5, K_0, K_3, K_4, K_6, K_7, K_8, K_9, K_<, K_>, K_?, K_A, K_B, K_BACK, K_BREAK, K_C, K_CAPS, K_D, K_DEL, K_DOWN, K_E, K_ESC, K_F, K_G, K_H, K_I, K_J, K_K, K_L, K_LEFT, K_LEFTALT, K_LEFTMETA, K_LINE, K_M, K_N, K_NOSCL, K_O, K_P, K_PIPE, K_PLUS, K_Q, K_QUOTE, K_R, K_RIGHT, K_RIGHTALT, K_RIGHTMETA, K_S, K_SEMI, K_T, K_TAB, K_TILDE, K_U, K_UP, K_USCORE, K_V, K_W, K_X, K_Y, K_Z, K_{, K_}: 1U_PAD, SiliconeSwitches:1U_PAD
- added K_CONTROL, K_LSHIFT, K_RSHIFT, K_SETUP: 2U_PAD, SiliconeSwitches:2U_PAD
- added K_RETURN: RETURN_PAD, SiliconeSwitches:RETURN_PAD
- added K_SPACE: SPACE_PAD, SiliconeSwitches:SPACE_PAD
- added SHIFT, SHIFT2, SPACE, \|: KEYSWITCH-PLAIN-MX-1U, Keyboard:KEYSWITCH-PLAIN-MX-1U
Connections:
- net KEYCOLUM0: now also K_7.P$2, K_<.P$2, K_ESC.P$2, K_G.P$2, K_J.P$2, K_NOSCL.P$2, K_RIGHTALT.P$2, K_SETUP.P$2, K_TAB.P$2, K_U.P$2; no longer 7.P0, ALT2.P0, COMMA.P0, ESC.P0, G.P0, J.P0, J1.7, J2.15, NO.P0, SETUP.P0, TAB.P0, U.P0
- net KEYCOLUM1: now also K-1.P$2, K_8.P$2, K_CAPS.P$2, K_H.P$2, K_I.P$2, K_K.P$2, K_LSHIFT.P$2, K_Q.P$2, K_RIGHTMETA.P$2; no longer 1.P0, 8.P0, CAPS.P0, H.P0, I.P0, J1.6, J2.14, K.P0, LEFTSHIFT.P0, META2.P0, Q.P0
- net KEYCOLUM2: now also K-2.P$2, K_0.P$2, K_9.P$2, K_>.P$2, K_CONTROL.P$2, K_L.P$2, K_LEFTMETA.P$2, K_O.P$2, K_W.P$2, K_Z.P$2; no longer 0.P0, 2.P0, 9.P0, CTRL.P0, J1.5, J2.13, L.P0, META.P0, O.P0, PERIOD.P0, W.P0, Z.P0
- net KEYCOLUM3: now also K_3.P$2, K_?.P$2, K_A.P$2, K_E.P$2, K_LEFT.P$2, K_LEFTALT.P$2, K_P.P$2, K_SEMI.P$2, K_USCORE.P$2, K_X.P$2; no longer 3.P0, ?/.P0, A.P0, ALT.P0, E.P0, J1.4, J2.12, KP_DASH.P0, LEFT.P0, P.P0, SEMI.P0, X.P0
- net KEYCOLUM4: now also K_4.P$2, K_C.P$2, K_DOWN.P$2, K_PLUS.P$2, K_QUOTE.P$2, K_R.P$2, K_RSHIFT.P$2, K_S.P$2, K_SPACE.P$2, K_{.P$2; no longer 4.P0, C.P0, DOWN.P0, EQUAL.P0, J1.3, J2.11, LBRACKET.P0, QUOTE.P0, R.P0, RIGHTSHIFT.P0, S.P0, SPACE1.P0, SPACE2.P0, SPACE3.P0
- net KEYCOLUM5: now also K-5.P$2, K_D.P$2, K_N.P$2, K_PIPE.P$2, K_RETURN.P$2, K_T.P$2, K_TILDE.P$2, K_UP.P$2, K_V.P$2, K_}.P$2; no longer 5.P0, D.P0, GRAVE.P0, J1.2, J2.10, N.P0, PIPE.P0, RBRACKET.P0, RETURN.P0, RETURN2.P0, T.P0, UP.P0, V.P0
- net KEYCOLUM6: now also K_6.P$2, K_B.P$2, K_BACK.P$2, K_BREAK.P$2, K_DEL.P$2, K_F.P$2, K_LINE.P$2, K_M.P$2, K_RIGHT.P$2, K_Y.P$2; no longer 6.P0, B.P0, BACK.P0, BRK.P0, DEL.P0, F.P0, J1.1, J2.9, LINE.P1, M.P0, RIGHT.P0, Y.P0
- net KEYROW0: now also K-1.P$1, K-2.P$1, K-5.P$1, K_3.P$1, K_4.P$1, K_6.P$1, K_ESC.P$1; no longer 1.P1, 2.P1, 3.P1, 4.P1, 5.P1, 6.P1, ESC.P1, J1.17, J3.15
- net KEYROW1: now also K_E.P$1, K_Q.P$1, K_R.P$1, K_SETUP.P$1, K_T.P$1, K_W.P$1, K_Y.P$1; no longer E.P1, J1.16, J3.14, Q.P1, R.P1, SETUP.P1, T.P1, W.P1, Y.P1
- net KEYROW2: now also K_A.P$1, K_CAPS.P$1, K_CONTROL.P$1, K_D.P$1, K_F.P$1, K_S.P$1, K_TAB.P$1; no longer A.P1, CAPS.P1, CTRL.P1, D.P1, F.P1, J1.15, J3.13, S.P1, TAB.P1
- net KEYROW3: now also K_B.P$1, K_C.P$1, K_LSHIFT.P$1, K_NOSCL.P$1, K_V.P$1, K_X.P$1, K_Z.P$1; no longer B.P1, C.P1, J1.14, J3.12, LEFTSHIFT.P1, NO.P1, V.P1, X.P1, Z.P1
- net KEYROW4: now also K_LEFTALT.P$1, K_LEFTMETA.P$1, K_M.P$1, K_N.P$1, K_RIGHTALT.P$1, K_RIGHTMETA.P$1, K_SPACE.P$1; no longer ALT.P1, ALT2.P1, J1.13, J3.11, M.P1, META.P1, META2.P1, N.P1, SPACE1.P1, SPACE2.P1, SPACE3.P1
- net KEYROW5: now also K_7.P$1, K_8.P$1, K_9.P$1, K_DOWN.P$1, K_LEFT.P$1, K_RIGHT.P$1, K_UP.P$1; no longer 7.P1, 8.P1, 9.P1, DOWN.P1, J1.12, J3.10, LEFT.P1, RIGHT.P1, UP.P1
- net KEYROW6: now also K_0.P$1, K_BACK.P$1, K_I.P$1, K_PLUS.P$1, K_TILDE.P$1, K_U.P$1, K_USCORE.P$1; no longer 0.P1, BACK.P1, EQUAL.P1, GRAVE.P1, I.P1, J1.11, J3.9, KP_DASH.P1, U.P1
- net KEYROW7: now also K_BREAK.P$1, K_G.P$1, K_H.P$1, K_O.P$1, K_P.P$1, K_{.P$1, K_}.P$1; no longer BRK.P1, G.P1, H.P1, J1.10, J3.8, LBRACKET.P1, O.P1, P.P1, RBRACKET.P1
- net KEYROW8: now also K_DEL.P$1, K_J.P$1, K_K.P$1, K_L.P$1, K_QUOTE.P$1, K_RETURN.P$1, K_SEMI.P$1; no longer DEL.P1, J.P1, J1.9, J3.7, K.P1, L.P1, QUOTE.P1, RETURN.P1, RETURN2.P1, SEMI.P1
- net KEYROW9: now also K_<.P$1, K_>.P$1, K_?.P$1, K_LINE.P$1, K_PIPE.P$1, K_RSHIFT.P$1; no longer ?/.P1, COMMA.P1, J1.8, J3.6, LINE.P0, PERIOD.P1, PIPE.P1, RIGHTSHIFT.P1
Other:
- moved on the sheet: 0, 1, 2, 3, 4, 5, 6, 7, 8, 9, A, ALT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
